File: PCB/PCB_design/PCB_design.kicad_sch (KiCad schematic)
At the start: 55 parts, among them J1 Conn_01x01_Pin, J2 Conn_01x01_Pin, J3 Conn_01x01_Pin, J4 Conn_01x01_Pin, J5 Conn_01x01_Pin, J6 Conn_01x01_Pin, J7 Conn_02x04_Counter_Clockwise, J8 Conn_01x01_Pin, K1 Relay_SPST-NO, K2 Relay_SPST-NO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

Commit message: J7 femelle
Parts:
- J7: footprint Connector_PinHeader_2.54mm:PinHeader_2x04_P2.54mm_Vertical -> Connector_PinSocket_2.54mm:PinSocket_2x04_P2.54mm_Vertical
Changed lines of the file:
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@@
 			)
 		)
-		(property "Footprint" "Connector_PinHeader_2.54mm:PinHeader_2x04_P2.54mm_Vertical"
+		(property "Footprint" "Connector_PinSocket_2.54mm:PinSocket_2x04_P2.54mm_Vertical"
 			(at 129.54 83.82 0)
 			(effects

Commit message: Routage : séparation primaire/secondaire
Parts:
- C4: footprint Capacitor_SMD:C_0805_2012Metric -> Capacitor_SMD:C_1206_3216Metric
Changed lines of the file:
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@@
 			)
 		)
-		(property "Footprint" "Capacitor_SMD:C_0805_2012Metric"
+		(property "Footprint" "Capacitor_SMD:C_1206_3216Metric"
 			(at 140.6652 49.53 0)
 			(effects

Commit message: Modif footprint relais & refaçonnage
Parts:
- K1, K2, K3, K4: footprint Touch_Switch_Custom:FH17-1A2STLE-DC5V -> Touch_Switch_Custom:relay
Changed lines of the file:
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@@
 			)
 		)
-		(property "Footprint" "Touch_Switch_Custom:FH17-1A2STLE-DC5V"
+		(property "Footprint" "Touch_Switch_Custom:relay"
 			(at 179.07 76.2 0)
 			(effects
@@
 			)
 		)
-		(property "Footprint" "Touch_Switch_Custom:FH17-1A2STLE-DC5V"
+		(property "Footprint" "Touch_Switch_Custom:relay"
 			(at 233.68 123.19 0)
 			(effects
@@
 			)
 		)
-		(property "Footprint" "Touch_Switch_Custom:FH17-1A2STLE-DC5V"
+		(property "Footprint" "Touch_Switch_Custom:relay"
 			(at 233.68 76.2 0)
 			(effects
@@
 			)
 		)
-		(property "Footprint" "Touch_Switch_Custom:FH17-1A2STLE-DC5V"
+		(property "Footprint" "Touch_Switch_Custom:relay"
 			(at 179.07 123.19 0)
 			(effects
