File: PCB/Control_card/Control_card.kicad_pcb (KiCad board)
At the start: 2 copper layers, 71.4 x 45.4 mm, 46 parts, among them IC1 TLSR8253F512ET48, J1 Conn_02x04_Counter_Clockwise, J2 Conn_01x01_Pin, J3 Conn_01x01_Pin, J4 Conn_01x01_Pin, J5 Conn_01x01_Pin, Y1 Crystal_GND24

Commit message: Routage
Routing:
- net 3.3V: track 288.4 -> 275.0 mm
- net CT1: track 22.3 -> 18.1 mm
- net CT3: track 24.8 -> 20.8 mm
- net VVD1V2: track 41.6 -> 38.1 mm
- net OutLed4: track 17.5 -> 14.2 mm
- net OutLed3: track 19.3 -> 16.8 mm
- net Net-(IC1-VANT): track 23.2 -> 21.1 mm, vias 4 -> 0
- net XC1: track 7.14 -> 8.13 mm
- net GND: track 74.8 -> 74.5 mm, vias 60 -> 59
- net ANT: vias 0 -> 4

Commit message: Rota IC contrôle
Parts:
- C15, C16, C17, C5, C7, C9, L2: moved to B.Cu
- moved C15 11.5 mm to (157.4, 77.0), turned to -90 degrees
- moved C5 11.3 mm to (148.1, 68.4), turned to 0 degrees
- moved C16 11.1 mm to (158.9, 77.0), turned to -90 degrees
- moved C17 8.72 mm to (154.0, 79.7), turned to -90 degrees
- moved C8 8.67 mm to (145.7, 70.3), turned to 90 degrees
- moved C6 8.24 mm to (142.7, 76.1), turned to -90 degrees
- moved L2 7.79 mm to (143.8, 72.8), turned to 90 degrees
- moved C4 6.08 mm to (144.2, 76.1), turned to -90 degrees
- moved C9 5.37 mm to (150.3, 78.9), turned to 0 degrees
- moved C7 4.86 mm to (147.2, 78.9), turned to 180 degrees
- moved L1 4.50 mm to (143.4, 78.8)
- moved C12 4.48 mm to (148.1, 78.8)
- moved C13 4.47 mm to (145.7, 79.6)
- moved C11 4.47 mm to (150.4, 79.6)
- moved L3 4.41 mm to (152.7, 78.8)
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Connections:
- IC1 pad 43: OutSw1 -> OutSw4
- IC1 pad 44: OutSw2 -> OutSw3
- IC1 pad 45: OutSw3 -> OutSw2
- IC1 pad 46: OutSw4 -> OutSw1
Routing:
- net GND: track 74.5 -> 5.82 mm, vias 59 -> 372
- net 3.3V: track 275.0 -> 240.9 mm, vias 16 -> 14
- net OutSw3: track 38.2 -> 13.9 mm, vias 6 -> 2
- net OutSw4: track 37.6 -> 13.6 mm, vias 6 -> 2
- net OutSw2: track 57.0 -> 33.6 mm, vias 6 -> 2
- net OutSw1: track 49.8 -> 33.3 mm
- net Net-(IC1-VANT): track 21.1 -> 4.72 mm
- net ANT: track 25.1 -> 12.7 mm, vias 4 -> 0
- net VVD1V2: track 38.1 -> 26.8 mm
- net XC2: track 8.20 -> 19.4 mm, vias 0 -> 4
- net XC1: track 8.13 -> 19.3 mm, vias 0 -> 4
- net In4: track 10.8 -> 19.9 mm
- net In3: track 12.4 -> 20.7 mm
- net In2: track 14.0 -> 21.5 mm
- net In1: track 15.7 -> 22.2 mm
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Other:
- outline, holes or cut-outs redrawn

Commit message: Ajout firmware
Parts:
- moved R1 1.75 mm to (150.7, 48.9)
- moved R2 1.38 mm to (150.7, 51.0)
- moved R3 0.99 mm to (150.7, 53.0)
- moved R4 0.61 mm to (150.7, 55.1)
- moved R5 0.33 mm to (150.8, 57.2)
Routing:
- net Net-(D1-A): track 3.11 -> 1.50 mm
- net OutLed1: track 22.2 -> 20.7 mm
- net OutLed2: track 21.8 -> 20.5 mm
- net Net-(D2-A): track 2.24 -> 1.50 mm
- net Net-(D3-A): track 2.09 -> 1.50 mm
Changed lines of the file:
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@@
 	(footprint "Resistor_SMD:R_0603_1608Metric"
 		(layer "F.Cu")
-		(at 150.490823 55.67631)
+		(at 150.7 55.1)
 		(descr "Resistor SMD 0603 (1608 Metric), square (rectangular) end terminal, IPC_7351 nominal, (Body size source: IPC-SM-782 page 72, https://www.pcb-3d.com/wordpress/wp-content/uploads/ipc-sm-782a_amendment_1_and_2.pdf), generated with kicad-footprint-generator")
 		(tags "resistor")
@@
 	(footprint "Resistor_SMD:R_0603_1608Metric"
 		(layer "F.Cu")
-		(at 150.490823 57.40351)
+		(at 150.75 57.2)
 		(descr "Resistor SMD 0603 (1608 Metric), square (rectangular) end terminal, IPC_7351 nominal, (Body size source: IPC-SM-782 page 72, https://www.pcb-3d.com/wordpress/wp-content/uploads/ipc-sm-782a_amendment_1_and_2.pdf), generated with kicad-footprint-generator")
 		(tags "resistor")
@@
 	(footprint "Resistor_SMD:R_0603_1608Metric"
 		(layer "F.Cu")
-		(at 150.541623 50.64711)
+		(at 150.7 48.9)
 		(descr "Resistor SMD 0603 (1608 Metric), square (rectangular) end terminal, IPC_7351 nominal, (Body size source: IPC-SM-782 page 72, https://www.pcb-3d.com/wordpress/wp-content/uploads/ipc-sm-782a_amendment_1_and_2.pdf), generated with kicad-footprint-generator")
 		(tags "resistor")
@@
 	(footprint "Resistor_SMD:R_0603_1608Metric"
 		(layer "F.Cu")
-		(at 150.516223 54.02531)
+		(at 150.7 53.05)
 		(descr "Resistor SMD 0603 (1608 Metric), square (rectangular) end terminal, IPC_7351 nominal, (Body size source: IPC-SM-782 page 72, https://www.pcb-3d.com/wordpress/wp-content/uploads/ipc-sm-782a_amendment_1_and_2.pdf), generated with kicad-footprint-generator")
 		(tags "resistor")
@@
 		(tags "capacitor")
 		(property "Reference" "C8"
-			(at 1.42 -1.51 270)
+			(at 1.42 -1.51 -90)
 			(layer "F.SilkS")
 			(effects
@@
 		)
 		(property "Value" "1u"
-			(at 0 1.43 270)
+			(at 0 1.43 -90)
 			(layer "F.Fab")
 			(effects
@@
 		)
 		(fp_text user "${REFERENCE}"
-			(at 0 0 270)
+			(at 0 0 -90)
 			(layer "F.Fab")
 			(effects
@@
 	(footprint "Resistor_SMD:R_0603_1608Metric"
 		(layer "F.Cu")
-		(at 150.541623 52.32351)
+		(at 150.7 50.95)
 		(descr "Resistor SMD 0603 (1608 Metric), square (rectangular) end terminal, IPC_7351 nominal, (Body size source: IPC-SM-782 page 72, https://www.pcb-3d.com/wordpress/wp-content/uploads/ipc-sm-782a_amendment_1_and_2.pdf), generated with kicad-footprint-generator")
 		(tags "resistor")
@@
 		(tags "capacitor")
 		(property "Reference" "C5"
-			(at 2.6 0 360)
+			(at 2.6 0 0)
 			(layer "B.SilkS")
 			(effects
@@
 		)
 		(property "Value" "1u"
-			(at 0 -1.43 360)
+			(at 0 -1.43 0)
 			(layer "B.Fab")
 			(effects
@@
 		)
 		(fp_text user "${REFERENCE}"
-			(at 0 0 360)
+			(at 0 0 0)
 			(layer "B.Fab")
 			(effects
@@
 		(tags "inductor")
 		(property "Reference" "L2"
-			(at 0.01 -1.86 270)
+			(at 0.01 -1.86 -90)
 			(layer "B.SilkS")
 			(effects
@@
 		)
 		(property "Value" "47u"
-			(at 0 -1.55 270)
+			(at 0 -1.55 -90)
 			(layer "B.Fab")
 			(effects
@@
 		)
 		(fp_text user "${REFERENCE}"
-			(at 0 0 270)
+			(at 0 0 -90)
 			(layer "B.Fab")
 			(effects
@@
 		(tags "capacitor")
 		(property "Reference" "C9"
-			(at -0.005 1.49 360)
+			(at -0.005 1.49 0)
 			(layer "B.SilkS")
 			(effects
@@
 		)
 		(property "Value" "1u"
-			(at 0 -1.43 360)
+			(at 0 -1.43 0)
 			(layer "B.Fab")
 			(effects
@@
 		)
 		(fp_text user "${REFERENCE}"
-			(at 0 0 360)
+			(at 0 0 0)
 			(layer "B.Fab")
 			(effects
@@
 	)
 	(segment
-		(start 154.998971 72.7025)
-		(end 154.195 72.7025)
+		(start 156.421373 72.399363)
+		(end 156.118236 72.7025)
 		(width 0.2)
 		(layer "F.Cu")
@@
 	)
 	(segment
-		(start 155.302108 72.399363)
-		(end 154.998971 72.7025)
+		(start 156.118236 72.7025)
+		(end 154.195 72.7025)
 		(width 0.2)
 		(layer "F.Cu")
@@
 	(segment
 		(start 157.76 72.399363)
-		(end 155.302108 72.399363)
+		(end 156.421373 72.399363)
 		(width 0.2)
 		(layer "F.Cu")
@@
 	)
 	(segment
-		(start 149.716623 52.32351)
-		(end 149.000823 52.32351)
+		(start 135.004333 48.28)
+		(end 133.560823 49.72351)
 		(width 0.2)
 		(layer "F.Cu")
@@
 	)
 	(segment
-		(start 148.32 48.28)
-		(end 135.004333 48.28)
+		(start 133.560823 49.72351)
+		(end 133.560823 51.13351)
 		(width 0.2)
 		(layer "F.Cu")
@@
 	)
 	(segment
-		(start 133.560823 49.72351)
-		(end 133.560823 51.13351)
+		(start 149.2 50.95)
+		(end 148.780823 50.530823)
 		(width 0.2)
 		(layer "F.Cu")
@@
 	)
 	(segment
-		(start 135.004333 48.28)
-		(end 133.560823 49.72351)
+		(start 148.780823 50.530823)
+		(end 148.780823 48.740823)
 		(width 0.2)
 		(layer "F.Cu")
@@
 	)
 	(segment
-		(start 149.000823 52.32351)
-		(end 148.780823 52.10351)
+		(start 149.875 50.95)
+		(end 149.2 50.95)
 		(width 0.2)
 		(layer "F.Cu")
@@
 	)
 	(segment
-		(start 148.780823 52.10351)
-		(end 148.780823 48.740823)
+		(start 148.32 48.28)
+		(end 135.004333 48.28)
 		(width 0.2)
 		(layer "F.Cu")
@@
 	)
 	(segment
-		(start 148.382623 54.02531)
-		(end 148.380823 54.02351)
-		(width 0.2)
-		(layer "F.Cu")
-		(net 47)
-	)
-	(segment
-		(start 149.691223 54.02531)
-		(end 148.382623 54.02531)
+		(start 148.35 53.05)
+		(end 149.875 53.05)
 		(width 0.2)
 		(layer "F.Cu")
@@
 	)
 	(via
-		(at 148.380823 54.02351)
+		(at 148.35 53.05)
 		(size 0.6)
 		(drill 0.3)
@@
 	)
 	(segment
-		(start 148.380823 53.944981)
-		(end 148.380823 54.02351)
+		(start 136.04149 49.08351)
+		(end 135.325 49.8)
 		(width 0.2)
 		(layer "B.Cu")
@@
 	)
 	(segment
-		(start 136.04149 49.08351)
-		(end 143.519352 49.08351)
+		(start 143.519352 49.08351)
+		(end 136.04149 49.08351)
 		(width 0.2)
 		(layer "B.Cu")
@@
 	)
 	(segment
-		(start 143.519352 49.08351)
-		(end 148.380823 53.944981)
+		(start 148.35 53.05)
+		(end 147.485842 53.05)
 		(width 0.2)
 		(layer "B.Cu")
@@
 	)
 	(segment
-		(start 135.325 49.8)
-		(end 136.04149 49.08351)
+		(start 147.485842 53.05)
+		(end 143.519352 49.08351)
 		(width 0.2)
 		(layer "B.Cu")
@@
 	)
 	(segment
-		(start 148.333623 55.67631)
-		(end 148.330823 55.67351)
+		(start 149.875 55.1)
+		(end 149.30149 55.67351)
 		(width 0.2)
 		(layer "F.Cu")
@@
 	)
 	(segment
-		(start 149.665823 55.67631)
-		(end 148.333623 55.67631)
+		(start 149.30149 55.67351)
+		(end 148.330823 55.67351)
 		(width 0.2)
 		(layer "F.Cu")
@@
 	)
 	(segment
-		(start 132.160823 49.76351)
-		(end 132.160823 51.13351)
+		(start 149.53 47.88)
+		(end 134.044333 47.88)
 		(width 0.2)
 		(layer "F.Cu")
@@
 	)
 	(segment
-		(start 149.28 47.88)
-		(end 134.044333 47.88)
+		(start 134.044333 47.88)
+		(end 132.160823 49.76351)
 		(width 0.2)
 		(layer "F.Cu")
@@
 	)
 	(segment
-		(start 149.716623 50.64711)
-		(end 149.716623 48.316623)
+		(start 132.160823 49.76351)
+		(end 132.160823 51.13351)
 		(width 0.2)
 		(layer "F.Cu")
@@
 	)
 	(segment
-		(start 134.044333 47.88)
-		(end 132.160823 49.76351)
+		(start 149.875 48.225)
+		(end 149.53 47.88)
 		(width 0.2)
 		(layer "F.Cu")
@@
 	)
 	(segment
-		(start 149.716623 48.316623)
-		(end 149.28 47.88)
+		(start 149.875 48.9)
+		(end 149.875 48.225)
 		(width 0.2)
 		(layer "F.Cu")
@@
 	)
 	(segment
-		(start 145.210823 56.68351)
-		(end 147.590823 56.68351)
+		(start 147.590823 56.68351)
+		(end 148.107313 57.2)
 		(width 0.2)
 		(layer "F.Cu")
@@
 	)
 	(segment
-		(start 148.310823 57.40351)
-		(end 149.665823 57.40351)
+		(start 145.210823 56.68351)
+		(end 147.590823 56.68351)
 		(width 0.2)
 		(layer "F.Cu")
@@
 	)
 	(segment
-		(start 147.590823 56.68351)
-		(end 148.310823 57.40351)
+		(start 148.107313 57.2)
+		(end 149.925 57.2)
 		(width 0.2)
 		(layer "F.Cu")
@@
 	)
 	(segment
-		(start 151.366623 49.358377)
-		(end 151.366623 50.64711)
+		(start 153.0125 48.925)
+		(end 151.8 48.925)
 		(width 0.2)
 		(layer "F.Cu")
@@
 	)
 	(segment
-		(start 151.8 48.925)
-		(end 151.366623 49.358377)
+		(start 151.775 48.9)
+		(end 151.525 48.9)
 		(width 0.2)
 		(layer "F.Cu")
@@
 	)
 	(segment
-		(start 153.0125 48.925)
-		(end 151.8 48.925)
+		(start 151.8 48.925)
+		(end 151.775 48.9)
 		(width 0.2)
 		(layer "F.Cu")
@@
 	(segment
 		(start 153.0125 50.975)
-		(end 153.0125 51.0375)
+		(end 151.55 50.975)
 		(width 0.2)
 		(layer "F.Cu")
@@
 	)
 	(segment
-		(start 153.0125 51.0375)
-		(end 151.72649 52.32351)
-		(width 0.2)
-		(layer "F.Cu")
-		(net 59)
-	)
-	(segment
-		(start 151.72649 52.32351)
-		(end 151.366623 52.32351)
+		(start 151.55 50.975)
+		(end 151.525 50.95)
 		(width 0.2)
 		(layer "F.Cu")
@@
 	(segment
 		(start 153.0125 53.025)
-		(end 152.625 53.025)
-		(width 0.2)
-		(layer "F.Cu")
-		(net 60)
-	)
-	(segment
-		(start 151.62469 54.02531)
-		(end 151.341223 54.02531)
+		(end 151.55 53.025)
 		(width 0.2)
 		(layer "F.Cu")
@@
 	)
 	(segment
-		(start 152.625 53.025)
-		(end 151.62469 54.02531)
+		(start 151.55 53.025)
+		(end 151.525 53.05)
 		(width 0.2)
 		(layer "F.Cu")
@@
 	)
 	(segment
-		(start 152.4 55.075)
-		(end 151.79869 55.67631)
+		(start 152.9875 55.1)
+		(end 151.525 55.1)
 		(width 0.2)
 		(layer "F.Cu")
@@
 	(segment
 		(start 153.0125 55.075)
-		(end 152.4 55.075)
+		(end 152.9875 55.1)
 		(width 0.2)
 		(layer "F.Cu")
@@
 	)
 	(segment
-		(start 151.79869 55.67631)
-		(end 151.315823 55.67631)
-		(width 0.2)
-		(layer "F.Cu")
-		(net 61)
-	)
-	(segment
-		(start 152.83399 57.40351)
-		(end 151.315823 57.40351)
-		(width 0.2)
-		(layer "F.Cu")
-		(net 62)
-	)
-	(segment
 		(start 153.0375 57.2)
-		(end 152.83399 57.40351)
+		(end 151.575 57.2)
 		(width 0.2)
 		(layer "F.Cu")
